File: single_esc.kicad_sch (KiCad schematic)
At the start: 37 parts, among them T201 BC847, T202 BC847, T203 BC847, U201 EFM8BB10

Commit message: cleaning up schematic
Parts:
- renumbered BL_TX201 to BL_TX1, C201 to C5, C202 to C6, C203 to C7, C204 to C8, FET201 to FET1, FET202 to FET2, FET203 to FET3, OUT_A201 to OUT_A1, OUT_B201 to OUT_B1, OUT_C201 to OUT_C1, R201 to R1, R219 to R10, R214 to R11, R202 to R12, R203 to R13, R204 to R14, R205 to R15, R206 to R16, R207 to R17, R208 to R18, R209 to R19, R220 to R2, R210 to R20, R211 to R3, R212 to R4, R213 to R5, R215 to R6, R216 to R7, R217 to R8, R218 to R9, T201 to T1, T202 to T2, T203 to T3, TP203 to TP7, TP202 to TP8, U201 to U2
